Commit message: Get real robot working (probably)

File: description/my_ros2_control_humble.xacro (robot description, xacro)
@@ -1,33 +1,32 @@
 <?xml version="1.0"?>
 <robot xmlns:xacro="http://www.ros.org/wiki/xacro">
+  <xacro:macro name="diffbot_ros2_control" params="name prefix">
     <xacro:unless value="$(arg sim_mode)">
-        <ros2_control name="RealRobot" type="system">
-            <hardware>
-                <plugin>diffdrive_arduino/DiffDriveArduinoHardware</plugin>
-                <param name="left_wheel_name">left_wheel_joint</param>
-                <param name="right_wheel_name">right_wheel_joint</param>
-                <param name="loop_rate">30</param>
-                <param name="device">/dev/ttyUSB0</param>
-                <param name="baud_rate">57600</param>
-                <param name="timeout_ms">1000</param>
-                <param name="enc_counts_per_rev">400</param>
-            </hardware>
-            <joint name="left_wheel_joint">
-                <command_interface name="velocity">
-                    <param name="min">-10</param>
-                    <param name="max">10</param>
-                </command_interface>
-                <state_interface name="position"/>
-                <state_interface name="velocity"/>
-            </joint>
-            <joint name="right_wheel_joint">
-                <command_interface name="velocity">
-                    <param name="min">-10</param>
-                    <param name="max">10</param>
-                </command_interface>
-                <state_interface name="position"/>
-                <state_interface name="velocity"/>
-            </joint>
-        </ros2_control>
+      <ros2_control name="${name}" type="system">
+        <hardware>
+          <plugin>diffdrive_arduino/DiffDriveArduinoHardware</plugin>
+          <param name="left_wheel_name">left_wheel_joint</param>
+          <param name="right_wheel_name">right_wheel_joint</param>
+          <param name="loop_rate">30</param>
+          <param name="device">/dev/ttyUSB0</param>
+          <param name="baud_rate">57600</param>
+          <param name="timeout_ms">1000</param>
+          <param name="enc_counts_per_rev">400</param>
+          <param name="pid_p">20</param>
+          <param name="pid_d">12</param>
+          <param name="pid_i">0</param>
+          <param name="pid_o">50</param>
+        </hardware>
+        <joint name="${prefix}left_wheel_joint">
+          <command_interface name="velocity"/>
+          <state_interface name="position"/>
+          <state_interface name="velocity"/>
+        </joint>
+        <joint name="${prefix}right_wheel_joint">
+          <command_interface name="velocity"/>
+          <state_interface name="position"/>
+          <state_interface name="velocity"/>
+        </joint>
+      </ros2_control>
     </xacro:unless>
     <xacro:if value="$(arg sim_mode)">
@@ -60,3 +59,4 @@
         </plugin>
     </gazebo>
+  </xacro:macro>
 </robot>
