Commit message: Solving bug rsp and failed to load ros2_control

File: description/camera.xacro (robot description, xacro)
@@ -1,6 +1,4 @@
 <?xml version="1.0"?>
 <robot xmlns:xacro="http://www.ros.org/wiki/xacro" >
-<<<<<<< HEAD
-<<<<<<< HEAD
     <!-- <joint name="camera_joint" type="fixed">
         <parent link="chassis"/>
@@ -81,18 +79,6 @@
         <child link="camera_link_optical"/>
         <origin xyz="0.025 0 0" rpy="0 ${pi/2} 0"/>
-=======
-        <origin xyz="0 0 0" rpy="${-pi/2} 0 ${-pi/2}"/>
->>>>>>> origin/main
-=======
-        <origin xyz="0 0 0" rpy="${-pi/2} 0 ${-pi/2}"/>
->>>>>>> origin/main
     </joint>
     <link name="camera_link_optical"></link>
-<<<<<<< HEAD
-<<<<<<< HEAD
-=======
->>>>>>> origin/main
-=======
->>>>>>> origin/main
     <gazebo reference="camera_link">
         <material>Gazebo/Black</material>

File: description/gazebo_control.xacro (robot description, xacro)
@@ -6,16 +6,6 @@
             <left_joint>left_wheel_joint</left_joint>
             <right_joint>right_wheel_joint</right_joint>
-<<<<<<< HEAD
-<<<<<<< HEAD
-            <wheel_separation>0.35</wheel_separation>
-            <wheel_diameter>0.1</wheel_diameter>
-=======
             <wheel_separation>0.297</wheel_separation>
             <wheel_diameter>0.066</wheel_diameter>
->>>>>>> origin/main
-=======
-            <wheel_separation>0.297</wheel_separation>
-            <wheel_diameter>0.066</wheel_diameter>
->>>>>>> origin/main
             <!-- Limits -->
             <max_wheel_torque>200</max_wheel_torque>

File: description/lidar.xacro (robot description, xacro)
@@ -4,13 +4,5 @@
         <parent link="chassis"/>
         <child link="laser_frame"/>
-<<<<<<< HEAD
-<<<<<<< HEAD
-        <origin xyz="-0.25 0.15 0.52" rpy="0 0 ${pi}"/>
-=======
         <origin xyz="0.122 0 0.212" rpy="0 0 0"/>
->>>>>>> origin/main
-=======
-        <origin xyz="0.122 0 0.212" rpy="0 0 0"/>
->>>>>>> origin/main
     </joint>
     <link name="laser_frame">
@@ -22,6 +14,4 @@
         </visual>
         <visual>
-<<<<<<< HEAD
-<<<<<<< HEAD
             <origin xyz="0 0 0.04"/>
             <geometry>
@@ -29,7 +19,4 @@
             </geometry>
             <material name="gray"/>
-=======
-=======
->>>>>>> origin/main
             <origin xyz="0 0 -0.05"/>
             <geometry>
@@ -37,8 +24,4 @@
             </geometry>
             <material name="black"/>
-<<<<<<< HEAD
->>>>>>> origin/main
-=======
->>>>>>> origin/main
         </visual>
         <collision>

File: description/my_camera.xacro (robot description, xacro)
@@ -46,4 +46,8 @@
             </camera>
             <plugin name="camera_controller" filename="libgazebo_ros_camera.so">
+                <ros>
+                    <remapping>~/image_raw:=/camera/image_raw</remapping>
+                    <remapping>~/camera_info:=/camera/camera_info</remapping>
+                </ros>
                 <frame_name>camera_link_optical</frame_name>
             </plugin>

File: description/my_lidar.xacro (robot description, xacro)
@@ -53,5 +53,5 @@
             <plugin name="laser_controller" filename="libgazebo_ros_ray_sensor.so">
                 <ros>
-                    <argument>~/out:=scan</argument>
+                    <remapping>~/out:=scan</remapping>
                 </ros>
                 <output_type>sensor_msgs/LaserScan</output_type>

File: description/myy_robot_core.xacro (robot description, xacro)
@@ -1,5 +1,5 @@
 <?xml version="1.0"?>
 <robot xmlns:xacro="http://www.ros.org/wiki/xacro" >
-    <xacro:include filename="inertial_macros.xacro"/>
+    <xacro:include filename="my_inertial_macros.xacro"/>
     <xacro:property name="chassis_length" value="1.0"/>
     <xacro:property name="chassis_width" value="0.6"/>

File: description/robot.urdf.xacro (robot description, xacro)
@@ -10,10 +10,4 @@
         <xacro:include filename="gazebo_control.xacro" />
     </xacro:unless>
-<<<<<<< HEAD
-<<<<<<< HEAD
-=======
->>>>>>> origin/main
-=======
->>>>>>> origin/main
     <xacro:include filename="lidar.xacro" />
     <xacro:include filename="camera.xacro" />

File: description/robot_core.xacro (robot description, xacro)
@@ -16,11 +16,5 @@
     <xacro:property name="caster_wheel_offset_x" value="0.075"/>
     <xacro:property name="caster_wheel_offset_z" value="${wheel_offset_z - wheel_radius + caster_wheel_radius}"/>
-<<<<<<< HEAD
-<<<<<<< HEAD
     <xacro:property name="PI" value="3.14285714285714"/>
-=======
->>>>>>> origin/main
-=======
->>>>>>> origin/main
     <material name="white">
         <color rgba="1 1 1 1" />
@@ -80,13 +74,5 @@
         <parent link="base_link"/>
         <child link="left_wheel"/>
-<<<<<<< HEAD
-<<<<<<< HEAD
-        <origin xyz="0 ${wheel_offset_y} 0" rpy="-${PI/2} 0 0" />
-=======
         <origin xyz="0 ${wheel_offset_y} 0" rpy="-${pi/2} 0 0" />
->>>>>>> origin/main
-=======
-        <origin xyz="0 ${wheel_offset_y} 0" rpy="-${pi/2} 0 0" />
->>>>>>> origin/main
         <axis xyz="0 0 1"/>
     </joint>
@@ -114,13 +100,5 @@
         <parent link="base_link"/>
         <child link="right_wheel"/>
-<<<<<<< HEAD
-<<<<<<< HEAD
-        <origin xyz="0 ${-wheel_offset_y} 0" rpy="${PI/2} 0 0" />
-=======
         <origin xyz="0 ${-wheel_offset_y} 0" rpy="${pi/2} 0 0" />
->>>>>>> origin/main
-=======
-        <origin xyz="0 ${-wheel_offset_y} 0" rpy="${pi/2} 0 0" />
->>>>>>> origin/main
         <axis xyz="0 0 -1"/>
     </joint>
