Commit message: fix ros2 control spawner for launch_sim

File: description/myy_robot.urdf.xacro (robot description, xacro)
@@ -5,5 +5,5 @@
     <xacro:include filename="myy_robot_core.xacro" />
     <xacro:if value="$(arg use_ros2_control)">
-        <xacro:include filename="my_ros2_control_humble.xacro" />
+        <xacro:include filename="my_ros2_control.xacro" />
     </xacro:if>
     <xacro:unless value="$(arg use_ros2_control)">

File: description/myy_robot_core.xacro (robot description, xacro)
@@ -75,5 +75,5 @@
         <parent link="base_link"/>
         <child link="left_wheel"/>
-        <origin xyz="${-wheel_offset_x} ${-wheel_offset_y} ${-wheel_offset_z}" rpy="${-pi/2} 0 0" />
+        <origin xyz="${wheel_offset_x} ${wheel_offset_y} ${-wheel_offset_z}" rpy="${-pi/2} 0 0" />
         <axis xyz="0 0 1"/>
     </joint>
@@ -102,5 +102,5 @@
         <parent link="base_link"/>
         <child link="right_wheel"/>
-        <origin xyz="${-wheel_offset_x} ${wheel_offset_y} ${-wheel_offset_z}" rpy="${pi/2} 0 0" />
+        <origin xyz="${wheel_offset_x} ${-wheel_offset_y} ${-wheel_offset_z}" rpy="${pi/2} 0 0" />
         <axis xyz="0 0 -1"/>
     </joint>
