Commit message: Real robot settings

File: description/my_camera.xacro (robot description, xacro)
@@ -4,5 +4,5 @@
         <parent link="chassis"/>
         <child link="camera_link"/>
-        <origin xyz="-0.25 -0.1 0.52" rpy="0 ${pi/20} 0"/>
+        <origin xyz="-0.25 -0.1 0.52" rpy="0 0 -${pi/2}"/>
     </joint>
     <link name="camera_link">
@@ -24,5 +24,5 @@
         <parent link="camera_link"/>
         <child link="camera_link_optical"/>
-        <origin xyz="0.025 0 0" rpy="0 ${pi/2} 0"/>
+        <origin xyz="0.025 0 0" rpy="-${pi/2} 0 0"/>
     </joint>
     <link name="camera_link_optical"></link>

File: description/my_ros2_control.xacro (robot description, xacro)
@@ -11,6 +11,18 @@
                 <param name="baud_rate">57600</param>
                 <param name="timeout_ms">1000</param>
-                <param name="enc_counts_per_rev">400</param>
+                <param name="enc_counts_per_rev">1600</param>
             </hardware>
+            <!--
+            <hardware>
+                <plugin>camdrive_arduino/CamDriveArduinoHardware</plugin>
+                <param name="left_wheel_name">left_wheel_joint</param>
+                <param name="right_wheel_name">right_wheel_joint</param>
+                <param name="loop_rate">30</param>
+                <param name="device">/dev/ttyUSB0</param>
+                <param name="baud_rate">57600</param>
+                <param name="timeout_ms">1000</param>
+                <param name="enc_counts_per_rev">1600</param>
+            </hardware>
+            -->
             <joint name="left_wheel_joint">
                 <command_interface name="velocity">

Commit message: update v1.5

File: description/my_camera.xacro (robot description, xacro)
@@ -4,5 +4,5 @@
         <parent link="chassis"/>
         <child link="camera_link"/>
-        <origin xyz="-0.25 -0.1 0.52" rpy="0 0 -${pi/2}"/>
+        <origin xyz="-0.02 -0.07 0.36" rpy="0 0 -${pi/2}"/>
     </joint>
     <link name="camera_link">

File: description/my_lidar.xacro (robot description, xacro)
@@ -7,5 +7,5 @@
         <parent link="chassis"/>
         <child link="laser_frame"/>
-        <origin xyz="-0.25 0.1 0.52" rpy="0 0 ${pi}"/>
+        <origin xyz="-0.03 0.07 0.36" rpy="0 0 ${pi}"/>
     </joint>
     <link name="laser_frame">

File: description/my_ros2_control.xacro (robot description, xacro)
@@ -10,5 +10,5 @@
                 <param name="device">/dev/ttyUSB0</param>
                 <param name="baud_rate">57600</param>
-                <param name="timeout_ms">1000</param>
+                <param name="timeout_ms">33</param>
                 <param name="enc_counts_per_rev">1600</param>
             </hardware>

File: description/my_ros2_control_humble.xacro (robot description, xacro)
@@ -12,6 +12,6 @@
           <param name="baud_rate">57600</param>
           <param name="timeout_ms">1000</param>
-          <param name="enc_counts_per_rev">400</param>
-          <param name="pid_p">20</param>
+          <param name="enc_counts_per_rev">1600</param>
+          <param name="pid_p">10</param>
           <param name="pid_d">12</param>
           <param name="pid_i">0</param>

File: description/myy_robot_core.xacro (robot description, xacro)
@@ -2,8 +2,8 @@
 <robot xmlns:xacro="http://www.ros.org/wiki/xacro" >
     <xacro:include filename="my_inertial_macros.xacro"/>
-    <xacro:property name="chassis_length" value="1.0"/>
-    <xacro:property name="chassis_width" value="0.6"/>
-    <xacro:property name="chassis_height" value="0.36"/>
-    <xacro:property name="chassis_mass" value="1.0"/>
+    <xacro:property name="chassis_length" value="0.80"/>
+    <xacro:property name="chassis_width" value="0.65"/>
+    <xacro:property name="chassis_height" value="0.31"/>
+    <xacro:property name="chassis_mass" value="45.0"/>
     <xacro:property name="wheel_radius" value="0.19"/>
     <xacro:property name="wheel_thickness" value="0.15"/>
@@ -41,5 +41,5 @@
         <parent link="base_link"/>
         <child link="base_footprint"/>
-        <origin xyz="0 0 ${-wheel_radius-wheel_offset_z}" rpy="0 0 0"/>
+        <origin xyz="-0.46 0 ${-wheel_radius-wheel_offset_z}" rpy="0 0 0"/>
     </joint>
     <link name="base_footprint"></link>
@@ -48,5 +48,5 @@
         <parent link="base_link"/>
         <child link="chassis"/>
-        <origin xyz="${-wheel_offset_x} 0 ${-wheel_offset_z}"/>
+        <origin xyz="-0.085 0 ${-wheel_offset_z}"/>
     </joint>
     <link name="chassis">

Commit message: new bracket

File: description/my_camera.xacro (robot description, xacro)
@@ -4,25 +4,25 @@
         <parent link="chassis"/>
         <child link="camera_link"/>
-        <origin xyz="-0.02 -0.07 0.36" rpy="0 0 -${pi/2}"/>
+        <origin xyz="-0.02 0 0.34" rpy="0 0 0"/>
     </joint>
     <link name="camera_link">
         <visual>
             <geometry>
-                <box size="0.1 0.07 0.1"/>
+                <box size="0.05 0.1 0.08"/>
             </geometry>
-            <material name="black"/>
-        </visual>
-        <visual>
-            <origin xyz="0.05 0 0" rpy="0 ${pi/2} 0"/>
-            <geometry>
-                <cylinder radius="0.02" length="0.01"/>
-            </geometry>
-            <material name="white"/>
+            <material name="gray"/>
         </visual>
     </link>
+<!--
+    <joint name="camera_o_joint" type="fixed">
+        <parent link="camera_link"/>
+        <child link="camera_o_link"/>
+        <origin xyz="0.02 0 0" rpy="-${pi/2} 0 0"/>
+    </joint>
+    <link name="camera_o_link"></link> -->
     <joint name="camera_optical_joint" type="fixed">
         <parent link="camera_link"/>
         <child link="camera_link_optical"/>
-        <origin xyz="0.025 0 0" rpy="-${pi/2} 0 0"/>
+        <origin xyz="0.02 0 0" rpy="-${pi/2} 0 -${pi/2}"/>
     </joint>
     <link name="camera_link_optical"></link>

File: description/my_lidar.xacro (robot description, xacro)
@@ -7,5 +7,5 @@
         <parent link="chassis"/>
         <child link="laser_frame"/>
-        <origin xyz="-0.03 0.07 0.36" rpy="0 0 ${pi}"/>
+        <origin xyz="-0.03 0 0.4" rpy="0 0 ${pi}"/>
     </joint>
     <link name="laser_frame">
